File: shield.sch (EAGLE design)
At the start: 12 parts

Commit message: Mirrored design to match header on FPGA
Parts:
- removed J4: (no value), SparkFun-Connectors:CONN_02
- added J0: (no value), SparkFun-Connectors:CONN_13X22X13
- J2: device SparkFun-Connectors:CONN_13X22X13 -> SparkFun-Connectors:CONN_02
- renumbered J3 to J1, R5 to R2, R_LOAD to R1
Connections:
- net GND: now also J0.26, J2.1; no longer J2.26, J4.1
- net N$1: now also J0.2; no longer J2.2
- net N$10: now also J0.15, SV1-2.S; no longer J2.15, SV1-4.S
- net N$11: now also J0.13; no longer J2.13
- net N$12: now also J0.11; no longer J2.11
- net N$2: now also J0.6; no longer J2.6
- net N$20: now also J0.9; no longer J2.9
- net N$3: now also J0.3; no longer J2.3
- net N$4: now also J0.16; no longer J2.16
- net N$5: now also J0.10; no longer J2.10
- net N$6: now also J0.12; no longer J2.12
- net N$7: now also J0.8, J2.2; no longer J2.8, J4.2
- net N$8: now also J0.14; no longer J2.14
- net N$9: now also J0.17, SV1-4.S; no longer J2.17, SV1-2.S
